Commit message: leapting_code

File: src/hzx/leapting_code/model_and_simulator/lt_gazebo/urdf/kuka3100_cover.urdf.xacro (robot description, xacro)
@@ -11,5 +11,5 @@
     <joint name="trailer" type="fixed">
         <!-- <origin xyz="2.3625 0.00117 -0.12" rpy="0 0 0" /> -->
-        <origin xyz="2.51565 0.00117 0.1505" rpy="0 0 0" />
+        <origin xyz="2.51565 0.00117 -0.0505" rpy="0 0 0" />
         <parent link="base_arm" />
         <child link="trailer" />
@@ -17,5 +17,5 @@
     <link name="base_link" />
     <joint name="base_link_arm" type="fixed">
-        <origin xyz="0 0 0.8" rpy="0 0 3.1415926" />
+        <origin xyz="0 0 1.254" rpy="0 0 3.1415926" />
         <parent link="base_link" />
         <child link="base_arm" />
