Commit message: update end_effector_pose

File: src/hzx/leapting_code/model_and_simulator/kr2700_moveit_config/config/gazebo_kr210r2700.urdf (robot description, URDF)
Before this commit: robot frontec_arm, 8 links, 7 joints
Links:
- link base_arm: geometry collision mesh filename=package://bringup/meshes/kr2700/base_arm.STL; visual mesh filename=package://bringup/meshes/kr2700/base_arm.STL
- link link_1: mass 0.01 -> 633.8; geometry collision mesh filename=package://bringup/meshes/kr2700/link_1.STL; visual mesh filename=package://bringup/meshes/kr2700/link_1.STL
- link link_2: mass 0.01 -> 691.94; geometry collision mesh filename=package://bringup/meshes/kr2700/link_2.STL; visual mesh filename=package://bringup/meshes/kr2700/link_2.STL
- link link_3: mass 0.01 -> 462.1; geometry collision mesh filename=package://bringup/meshes/kr2700/link_3.STL; visual mesh filename=package://bringup/meshes/kr2700/link_3.STL
- link link_4: mass 0.01 -> 39.417; geometry collision mesh filename=package://bringup/meshes/kr2700/link_4.STL; visual mesh filename=package://bringup/meshes/kr2700/link_4.STL
- link link_5: mass 0.01 -> 53.275; geometry collision mesh filename=package://bringup/meshes/kr2700/link_5.STL; visual mesh filename=package://bringup/meshes/kr2700/link_5.STL
- link link_6: mass 0.01 -> 4.4993; geometry collision mesh filename=package://bringup/meshes/kr2700/link_6.STL; visual mesh filename=package://bringup/meshes/kr2700/link_6.STL
- link tool0: mass 0.1 -> 0.01; geometry collision mesh filename=package://bringup/meshes/kr2700/tool.STL; visual mesh filename=package://bringup/meshes/kr2700/tool.STL
Joints:
- joint joint_a1: limit lower=-3.220132469929538 upper=3.2288591161895095 effort=100 velocity=1 -> lower=-3.220132469929538 upper=3.141592653589793 effort=100 velocity=1
- joint joint_a4: limit lower=-5.235987755982989 upper=6.1086523819801535 effort=100 velocity=1 -> lower=-3.141592653589793 upper=3.141592653589793 effort=100 velocity=1
- joint joint_a6: limit lower=-6.1086523819801535 upper=6.1086523819801535 effort=100 velocity=1 -> lower=-3.141592653589793 upper=3.141592653589793 effort=100 velocity=1

File: src/hzx/leapting_code/model_and_simulator/kr3100_moveit_config/config/gazebo_kr210r2700.urdf (robot description, URDF)
Before this commit: robot frontec_arm, 8 links, 7 joints
Links:
- link base_arm: geometry collision mesh filename=package://bringup/meshes/kr3100/base_arm.STL; visual mesh filename=package://bringup/meshes/kr3100/base_arm.STL
- link link_1: mass 0.01 -> 633.8; geometry collision mesh filename=package://bringup/meshes/kr3100/link_1.STL; visual mesh filename=package://bringup/meshes/kr3100/link_1.STL
- link link_2: mass 0.01 -> 691.94; geometry collision mesh filename=package://bringup/meshes/kr3100/link_2.STL; visual mesh filename=package://bringup/meshes/kr3100/link_2.STL
- link link_3: mass 0.01 -> 462.1; geometry collision mesh filename=package://bringup/meshes/kr3100/link_3.STL; visual mesh filename=package://bringup/meshes/kr3100/link_3.STL
- link link_4: mass 0.01 -> 39.417; geometry collision mesh filename=package://bringup/meshes/kr3100/link_4.STL; visual mesh filename=package://bringup/meshes/kr3100/link_4.STL
- link link_5: mass 0.01 -> 53.275; geometry collision mesh filename=package://bringup/meshes/kr3100/link_5.STL; visual mesh filename=package://bringup/meshes/kr3100/link_5.STL
- link link_6: mass 0.01 -> 4.4993; geometry collision mesh filename=package://bringup/meshes/kr3100/link_6.STL; visual mesh filename=package://bringup/meshes/kr3100/link_6.STL
- link tool0: mass 0.1 -> 0.01; geometry collision mesh filename=package://bringup/meshes/kr3100/tool.STL; visual mesh filename=package://bringup/meshes/kr3100/tool.STL
Joints:
- joint joint_a1: limit lower=-3.220132469929538 upper=3.2288591161895095 effort=100 velocity=1 -> lower=-3.220132469929538 upper=3.141592653589793 effort=100 velocity=1
- joint joint_a4: limit lower=-5.235987755982989 upper=6.1086523819801535 effort=100 velocity=1 -> lower=-3.141592653589793 upper=3.141592653589793 effort=100 velocity=1
- joint joint_a6: limit lower=-6.1086523819801535 upper=6.1086523819801535 effort=100 velocity=1 -> lower=-3.141592653589793 upper=3.141592653589793 effort=100 velocity=1
